File: eb-ground-station/power_board/ground_station_power_board/ground_station_power_board.sch (EAGLE design)
At the start: 0 parts

Commit message: progress on the power board
Parts:
- added C1, C5, C6, C7: 0.1uF, SparkFun-Capacitors:0.1UF-0603-25V-5%
- added C10, C4, C8, C9: 10uF, SparkFun-Capacitors:10UF-1206-6.3V-20%
- added C2: 100UF-CAP-EMVH630ARA101MKE0SCHEMI-KE0-M, GROUND-STATION-POWER-BOARD:100UF-CAP-EMVH630ARA101MKE0SCHEMI-KE0-M
- added C3: 4.7uF, SparkFun-Capacitors:4.7UF-1206-16V-(+80/-20%)
- added J1: CONN_20X2SHROUDED, SparkFun-Connectors:CONN_20X2SHROUDED
- added J2, J3: (no value), SparkFun-Connectors:CONN_03LONGPADS
- added R1, R2: 4.7k, SparkFun-Resistors:4.7KOHM-0603-1/10W-1%
- added R10, R11, R12, R4, R5, R6, R7, R8, R9: (no value), SparkFun-Resistors:RESISTOR0603
- added R3: 220, SparkFun-Resistors:RESISTOR0603
- added U$1, U$2, U$3, U$4, U$5, U$6: 1719031-PHONEIX-CONTACT-DBL-TERMINAL-BLOCK, GROUND-STATION-POWER-BOARD:1719031-PHONEIX-CONTACT-DBL-TERMINAL-BLOCK
- added U$10, U$11, U$12, U$13, U$14, U$16: SQJ459EP_MOSFET_P_CHAN, GROUND-STATION-POWER-BOARD:SQJ459EP_MOSFET_P_CHAN
- added U$15, U$17, U$18, U$8, U$9: DMN61D8LVT-DUAL-N-CHANNEL-MOSFET, GROUND-STATION-POWER-BOARD:DMN61D8LVT-DUAL-N-CHANNEL-MOSFET
- added U$7: 1714971-PHONEIX-CONTACT-TERMINAL-BLOCK, GROUND-STATION-POWER-BOARD:1714971-PHONEIX-CONTACT-TERMINAL-BLOCK
- added U1: ADS1115IDGSTDGS10-M, GROUND-STATION-POWER-BOARD:ADS1115IDGSTDGS10-M
- added U2: MCP23017T-E/SOSOIC28-W_MC-M, GROUND-STATION-POWER-BOARD:MCP23017T-E/SOSOIC28-W_MC-M
- added U3, U4, U5: MICROCHIP-TC427-MOSFET-DRIVERSOIC8, GROUND-STATION-POWER-BOARD:MICROCHIP-TC427-MOSFET-DRIVERSOIC8
- added U6: NCV1117ST33T3G, NCV1117ST33T3G:NCV1117ST33T3G
- added U7, U8, U9: EXB-A10P391JC_ARRAY_EXBA-M, temp-lib:EXB-A10P391JC_ARRAY_EXBA-M
Connections:
- new net 12V: C1.1, C10.1, C2.11, C4.1, C8.1, C9.1, U$10.S, U$11.S, U$12.S, U$13.S, U$14.S, U$16.S, U$7.1, U3.VDD, U4.VDD, U5.VDD, U6.INPUT, U9.55
- new net 3.3V: C3.1, C5.1, C6.1, C7.1, R1.2, R2.2, U1.VDD, U2.VDD, U6.OUTPUT
- new net GND: C1.2, C10.2, C2.22, C3.2, C4.2, C5.2, C6.2, C7.2, C8.2, C9.2, J1.14, J1.20, J1.25, J1.30, J1.34, J1.39, J1.6, J1.9, U$15.S1, U$15.S2, U$17.S1, U$17.S2, U$18.S1, U$18.S2, U$7.2, U$8.S1, U$8.S2, U$9.S1, U$9.S2, U1.GND, U2.!RESET, U2.GND, U3.GND, U4.GND, U5.GND, U6.ADJUST/GROUND, U7.55, U8.55
- new net N$1: R3.1
- new net N$10: R12.1
- new net N$2: R5.1
- new net N$21: R11.2, U$8.G1
- new net N$23: R12.2, U$8.G2
- new net N$25: R6.2, U$17.G1
- new net N$26: R4.2, U$17.G2
- new net N$29: R7.2, U$15.G1
- new net N$3: R4.1
- new net N$30: R5.2, U$18.G1
- new net N$31: R8.2, U$15.G2
- new net N$32: R3.2, U$18.G2
- new net N$33: R9.2, U$9.G1
- new net N$34: R10.2, U$9.G2
- new net N$4: R6.1
- new net N$5: R7.1
- new net N$6: R8.1
- new net N$7: R9.1
- new net N$8: R10.1
- new net N$9: R11.1
- new net OUT1: U2.GPA0, U8.66
- new net OUT10: U2.GPB1, U7.44
- new net OUT11: U2.GPB2, U7.77
- new net OUT12: U2.GPB3, U7.33
- new net OUT13: U2.GPB4, U7.88
- new net OUT14: U2.GPB5, U7.22
- new net OUT15: U2.GPB6, U7.99
- new net OUT16: U2.GPB7, U7.11
- new net OUT2: U2.GPA1, U8.44
- new net OUT3: U2.GPA2, U8.77
- new net OUT4: U2.GPA3, U8.33
- new net OUT5: U2.GPA4, U8.88
- new net OUT6: U2.GPA5, U8.22
- new net OUT7: U2.GPA6, U8.99
- new net OUT8: U2.GPA7, U8.11
- new net OUT9: U2.GPB0, U7.66
- new net PWR_FET_G1: U$16.G, U$8.D2, U9.11
- new net PWR_FET_G2: U$10.G, U$8.D1, U9.99
- new net PWR_FET_G3: U$11.G, U$9.D2, U9.22
- new net PWR_FET_G4: U$12.G, U$9.D1, U9.88
- new net PWR_FET_G5: U$13.G, U$15.D2, U9.33
- new net PWR_FET_G6: U$14.G, U$15.D1, U9.77
- new net PWR_P_FET_1: U$1.3, U$14.D
- new net PWR_P_FET_2: U$1.1, U$13.D
- new net PWR_P_FET_3: U$12.D, U$2.3
- new net PWR_P_FET_4: U$11.D, U$2.1
- new net PWR_P_FET_5: U$10.D, U$3.3
- new net PWR_P_FET_6: U$16.D, U$3.1
- new net RX_UART: J1.10
- new net SCL: J1.5, R2.1, U1.SCL, U2.SCL
- new net SDA: J1.3, R1.1, U1.SDA, U2.SDA
- new net TX_UART: J1.8
Other:
- note added: "SERIAL BUSES"
