File: eb-ground-station/power_board/ground_station_power_board/ground_station_power_board.sch (EAGLE design)
At the start: 52 parts, among them J1 CONN_20X2SHROUDED, U1 ADS1115IDGSTDGS10-M, U2 MCP23017T-E/SOSOIC28-W_MC-M, U3 MICROCHIP-TC427-MOSFET-DRIVER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, U4 MICROCHIP-TC427-MOSFET-DRIVER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, U5 MICROCHIP-TC427-MOSFET-DRIVER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, U6 NCV1117ST33T3G, U7 EXB-A10P391JC_ARRAY_EXBA-M, U8 EXB-A10P391JC_ARRAY_EXBA-M, U9 EXB-A10P391JC_ARRAY_EXBA-M

Commit message: Power board is mostly wrapped up
Parts:
- removed J2, J3: (no value), SparkFun-Connectors:CONN_03LONGPADS
- removed R10, R11, R12, R4, R5, R6, R7, R8, R9: (no value), SparkFun-Resistors:RESISTOR0603
- removed U5: MICROCHIP-TC427-MOSFET-DRIVERSOIC8, GROUND-STATION-POWER-BOARD:MICROCHIP-TC427-MOSFET-DRIVERSOIC8
- removed U6: NCV1117ST33T3G, NCV1117ST33T3G:NCV1117ST33T3G
- added D1, D10, D11, D12, D13, D14, D15, D16, D17, D2, D3, D4, D5, D6, D7, D8, D9: (no value), SparkFun-LED:LED0603
- added J4: (no value), SparkFun-Connectors:CONN_06LONGPADS
- added J5: (no value), SparkFun-Connectors:CONN_04LONGPADS
- added U$19, U$20, U$21, U$25, U$26, U$27, U$28: RES-ARRAY-742C083, GROUND-STATION-POWER-BOARD:RES-ARRAY-742C083
- added U$22, U$23, U$24: TC4427-FET-GATE-DRVR, GROUND-STATION-POWER-BOARD:TC4427-FET-GATE-DRVR
- R3: value 220 -> 800; device SparkFun-Resistors:RESISTOR0603 -> SparkFun-Resistors:4.7KOHM-0603-1/10W-1%
- U$7: value 1714971-PHONEIX-CONTACT-TERMINAL-BLOCK -> 1714955-PHONEIX-CONTACT-TERMINAL-BLOCK; device GROUND-STATION-POWER-BOARD:1714971-PHONEIX-CONTACT-TERMINAL-BLOCK -> GROUND-STATION-POWER-BOARD:1714955-PHONEIX-CONTACT-TERMINAL-BLOCK
- U2: value MCP23017T-E/SOSOIC28-W_MC-M -> MCP23017T-E/SOQFN; device GROUND-STATION-POWER-BOARD:MCP23017T-E/SOSOIC28-W_MC-M -> GROUND-STATION-POWER-BOARD:MCP23017T-E/SOQFN
- U3: value MICROCHIP-TC427-MOSFET-DRIVERSOIC8 -> MIC5239-3.3YMMMSOP-8_MM-M; device GROUND-STATION-POWER-BOARD:MICROCHIP-TC427-MOSFET-DRIVERSOIC8 -> GROUND-STATION-POWER-BOARD:MIC5239-3.3YMMMSOP-8_MM-M
- U4: value MICROCHIP-TC427-MOSFET-DRIVERSOIC8 -> MCP9808T-E/MCDFN8_2X3MC-M; device GROUND-STATION-POWER-BOARD:MICROCHIP-TC427-MOSFET-DRIVERSOIC8 -> GROUND-STATION-POWER-BOARD:MCP9808T-E/MCDFN8_2X3MC-M
Connections:
- removed net N$10: R12.1
- removed net N$21: R11.2, U$8.G1
- removed net N$23: R12.2, U$8.G2
- removed net N$25: R6.2, U$17.G1
- removed net N$30: R5.2, U$18.G1
- removed net N$31: R8.2, U$15.G2
- removed net N$32: R3.2, U$18.G2
- removed net N$33: R9.2, U$9.G1
- removed net N$34: R10.2, U$9.G2
- removed net N$5: R7.1
- removed net N$6: R8.1
- removed net N$7: R9.1
- removed net N$8: R10.1
- new net ADC1: U$5.3, U1.AIN3
- new net ADC2: U$5.1, U1.AIN2
- new net ADC3: U$6.3, U1.AIN1
- new net ADC4: U$6.1, U1.AIN0
- new net G1: U$21.!1OE6, U$8.G2
- new net G10: U$17.G1, U$20.!1OE4
- new net G2: U$21.!1OE8, U$8.G1
- new net G3: U$19.!1OE2, U$9.G2
- new net G4: U$19.!1OE4, U$9.G1
- new net G5: U$15.G2, U$19.!1OE6
- new net G6: U$15.G1, U$19.!1OE8
- new net G7: U$18.G2, U$20.!1OE6
- new net G8: U$18.G1, U$20.!1OE8
- new net G9: U$17.G2, U$20.!1OE2
- new net HIGH_OUT_1: U$24.A-OUT, U$3.4
- new net HIGH_OUT_2: U$24.B-OUT, U$3.2
- new net HIGH_OUT_3: U$1.4, U$23.A-OUT
- new net HIGH_OUT_4: U$1.2, U$23.B-OUT
- new net HIGH_OUT_5: U$2.4, U$22.A-OUT
- new net HIGH_OUT_6: U$2.2, U$22.B-OUT
- new net LOW_OUT_1: U$18.D2, U$4.3
- new net LOW_OUT_2: U$18.D1, U$4.4
- new net LOW_OUT_3: U$17.D2, U$4.2
- new net LOW_OUT_4: U$17.D1, U$4.1
- new net N$14: D6.A, U$26.!1OE8
- new net N$15: D7.A, U$26.!1OE6
- new net N$16: D8.A, U$26.!1OE4
- new net N$17: D9.A, U$26.!1OE2
- new net N$27: D11.A, U$27.!1OE6
- new net N$28: D12.A, U$27.!1OE4
- new net N$38: D14.A, U$28.!1OE8
- new net N$39: D15.A, U$28.!1OE6
- new net N$40: D16.A, U$28.!1OE4
- new net N$41: D17.A, U$28.!1OE2
- new net RX: J4.4
- new net TX: J4.5
- net 12V: now also D5.A, U$22.VDD, U$23.VDD, U$24.VDD, U3.EN, U3.IN; no longer U3.VDD, U4.VDD, U5.VDD, U6.INPUT
- net 3.3V: now also J4.3, J5.3, U3.OUT, U4.VDD; no longer U6.OUTPUT
- net GND: now also D1.C, D10.C, D11.C, D12.C, D13.C, D14.C, D15.C, D16.C, D17.C, D2.C, D3.C, D4.C, D6.C, D7.C, D8.C, D9.C, J4.1, J5.4, R3.2, U$22.GND, U$23.GND, U$24.GND, U$5.2, U$5.4, U$6.2, U$6.4, U1.ADDR, U2.A0, U2.A1, U2.A2, U4.A0, U4.A1, U4.A2; no longer U5.GND, U6.ADJUST/GROUND
- net N$1: now also D1.A, U$25.!1OE8; no longer R3.1
- net N$2: now also D2.A, U$25.!1OE6; no longer R5.1
- net N$26: now also D10.A, U$27.!1OE8; no longer R4.2, U$17.G2
- net N$29: now also D13.A, U$27.!1OE2; no longer R7.2, U$15.G1
- net N$3: now also D3.A, U$25.!1OE4; no longer R4.1
- net N$4: now also D4.A, U$25.!1OE2; no longer R6.1
- net N$9: now also D5.C, R3.1; no longer R11.1
- net OUT1: now also U$24.B-IN, U$26.!1OE5, U2.GPB2, U8.22; no longer U2.GPA0, U8.66
- net OUT10: now also U$20.!1OE1, U$27.!1OE5, U2.GPA6; no longer U2.GPB1
- net OUT11: now also U$19.!1OE3, U$28.!1OE7, U2.GPA3, U7.88; no longer U2.GPB2, U7.77
- net OUT12: now also U$19.!1OE7, U$27.!1OE3, U2.GPA5, U7.77; no longer U2.GPB3, U7.33
- net OUT13: now also U$19.!1OE5, U$27.!1OE1, U2.GPA4, U7.33; no longer U2.GPB4, U7.88
- net OUT14: now also U$19.!1OE1, U$28.!1OE5, U2.GPA2; no longer U2.GPB5
- net OUT15: now also U$21.!1OE7, U$28.!1OE3, U2.GPA1; no longer U2.GPB6
- net OUT16: now also U$21.!1OE5, U$28.!1OE1, U2.GPA0; no longer U2.GPB7
- net OUT2: now also U$24.A-IN, U$26.!1OE7, U2.GPB3, U8.88; no longer U2.GPA1, U8.44
- net OUT3: now also U$23.B-IN, U$25.!1OE5, U2.GPB6, U8.44; no longer U2.GPA2, U8.77
- net OUT4: now also U$23.A-IN, U$25.!1OE7, U2.GPB7, U8.66; no longer U2.GPA3, U8.33
- net OUT5: now also U$22.B-IN, U$25.!1OE1, U2.GPB4, U8.33; no longer U2.GPA4, U8.88
- net OUT6: now also U$22.A-IN, U$25.!1OE3, U2.GPB5, U8.77; no longer U2.GPA5, U8.22
- net OUT7: now also U$20.!1OE7, U$26.!1OE3, U2.GPB1; no longer U2.GPA6
- net OUT8: now also U$20.!1OE5, U$26.!1OE1, U2.GPB0; no longer U2.GPA7
- net OUT9: now also U$20.!1OE3, U$27.!1OE7, U2.GPA7; no longer U2.GPB0
- net PWR_FET_G1: now also U$10.G, U9.88; no longer U$16.G, U9.11
- net PWR_FET_G2: now also U$16.G, U9.22; no longer U$10.G, U9.99
- net PWR_FET_G3: now also U$12.G, U9.77; no longer U$11.G, U9.22
- net PWR_FET_G4: now also U$11.G, U9.33; no longer U$12.G, U9.88
- net PWR_FET_G5: now also U$14.G, U9.66; no longer U$13.G, U9.33
- net PWR_FET_G6: now also U$13.G, U9.44; no longer U$14.G, U9.77
- net SCL: now also J5.1, U4.SCL
- net SDA: now also J5.2, U4.SDA
Other:
- moved on the sheet: C1, C10, C2, C3, C4, C5, C6, C7, C8, C9, J1, R1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

Commit message: some final changes
Parts:
- removed U$10, U$11, U$12, U$13, U$14, U$16: SQJ459EP_MOSFET_P_CHAN, GROUND-STATION-POWER-BOARD:SQJ459EP_MOSFET_P_CHAN
- removed U$15, U$17, U$18, U$8, U$9: DMN61D8LVT-DUAL-N-CHANNEL-MOSFET, GROUND-STATION-POWER-BOARD:DMN61D8LVT-DUAL-N-CHANNEL-MOSFET
- removed U$19, U$20, U$21, U$25, U$26, U$27, U$28: RES-ARRAY-742C083, GROUND-STATION-POWER-BOARD:RES-ARRAY-742C083
- removed U$22, U$23, U$24: TC4427-FET-GATE-DRVR, GROUND-STATION-POWER-BOARD:TC4427-FET-GATE-DRVR
- removed U7, U8, U9: EXB-A10P391JC_ARRAY_EXBA-M, temp-lib:EXB-A10P391JC_ARRAY_EXBA-M
- added E1, E2: (no value), oresat-rcl:L-BEAD-0805-B
- added Q1, Q2, Q3, Q4, Q5, Q6: SQJ459EP_MOSFET_P_CHAN, GROUND-STATION-POWER-BOARD:SQJ459EP_MOSFET_P_CHAN
- added Q15, Q17, Q18, Q8, Q9: DMN61D8LVT-DUAL-N-CHANNEL-MOSFET, GROUND-STATION-POWER-BOARD:DMN61D8LVT-DUAL-N-CHANNEL-MOSFET
- added Q22, Q23, Q24: TC4427-FET-GATE-DRVR, GROUND-STATION-POWER-BOARD:TC4427-FET-GATE-DRVR
- added R10, R8, R9: EXB-A10P391JC_ARRAY_EXBA-M, temp-lib:EXB-A10P391JC_ARRAY_EXBA-M
- added R11, R12, R13: 220, GROUND-STATION-POWER-BOARD:RES-ARRAY-742C083
- added R4, R5, R6, R7: 680, GROUND-STATION-POWER-BOARD:RES-ARRAY-742C083
- C10, C4, C8, C9: device SparkFun-Capacitors:10UF-1206-6.3V-20% -> SparkFun-Capacitors:10UF-0805-10V-10%
- C2: value 100UF-CAP-EMVH630ARA101MKE0SCHEMI-KE0-M -> 100UF
- C3: value 4.7uF -> 10uF; device SparkFun-Capacitors:4.7UF-1206-16V-(+80/-20%) -> SparkFun-Capacitors:10UF-0805-10V-10%
- R3: value 800 -> 806
Connections:
- removed net RX: J4.4
- removed net TX: J4.5
- new net AGND: C6.2, E2.2, U$5.2, U$5.4, U$6.2, U$6.4, U1.ADDR, U1.ALERT/RDY, U1.GND
- new net N$5: C6.1, E1.1, U1.VDD
- net 12V: now also Q1.S, Q2.S, Q22.VDD, Q23.VDD, Q24.VDD, Q3.S, Q4.S, Q5.S, Q6.S, R10.55; no longer U$10.S, U$11.S, U$12.S, U$13.S, U$14.S, U$16.S, U$22.VDD, U$23.VDD, U$24.VDD, U9.55
- net 3.3V: now also E1.2; no longer C6.1, U1.VDD
- net G1: now also Q8.G2, R11.!1OE6; no longer U$21.!1OE6, U$8.G2
- net G10: now also Q17.G1, R13.!1OE4; no longer U$17.G1, U$20.!1OE4
- net G2: now also Q8.G1, R11.!1OE8; no longer U$21.!1OE8, U$8.G1
- net G3: now also Q9.G2, R12.!1OE2; no longer U$19.!1OE2, U$9.G2
- net G4: now also Q9.G1, R12.!1OE4; no longer U$19.!1OE4, U$9.G1
- net G5: now also Q15.G2, R12.!1OE6; no longer U$15.G2, U$19.!1OE6
- net G6: now also Q15.G1, R12.!1OE8; no longer U$15.G1, U$19.!1OE8
- net G7: now also Q18.G2, R13.!1OE6; no longer U$18.G2, U$20.!1OE6
- net G8: now also Q18.G1, R13.!1OE8; no longer U$18.G1, U$20.!1OE8
- net G9: now also Q17.G2, R13.!1OE2; no longer U$17.G2, U$20.!1OE2
- net GND: now also E2.1, Q15.S1, Q15.S2, Q17.S1, Q17.S2, Q18.S1, Q18.S2, Q22.GND, Q23.GND, Q24.GND, Q8.S1, Q8.S2, Q9.S1, Q9.S2, R8.55, R9.55; no longer C6.2, U$15.S1, U$15.S2, U$17.S1, U$17.S2, U$18.S1, U$18.S2, U$22.GND, U$23.GND, U$24.GND, U$5.2, U$5.4, U$6.2, U$6.4, U$8.S1, U$8.S2, U$9.S1, U$9.S2, U1.ADDR, U1.GND, U7.55, U8.55
- net HIGH_OUT_1: now also Q24.A-OUT; no longer U$24.A-OUT
- net HIGH_OUT_2: now also Q24.B-OUT; no longer U$24.B-OUT
- net HIGH_OUT_3: now also Q23.A-OUT; no longer U$23.A-OUT
- net HIGH_OUT_4: now also Q23.B-OUT; no longer U$23.B-OUT
- net HIGH_OUT_5: now also Q22.A-OUT; no longer U$22.A-OUT
- net HIGH_OUT_6: now also Q22.B-OUT; no longer U$22.B-OUT
- net LOW_OUT_1: now also Q18.D2; no longer U$18.D2
- net LOW_OUT_2: now also Q18.D1; no longer U$18.D1
- net LOW_OUT_3: now also Q17.D2; no longer U$17.D2
- net LOW_OUT_4: now also Q17.D1; no longer U$17.D1
- net N$1: now also R4.!1OE8; no longer U$25.!1OE8
- net N$14: now also R5.!1OE8; no longer U$26.!1OE8
- net N$15: now also R5.!1OE6; no longer U$26.!1OE6
- net N$16: now also R5.!1OE4; no longer U$26.!1OE4
- net N$17: now also R5.!1OE2; no longer U$26.!1OE2
- net N$2: now also R4.!1OE6; no longer U$25.!1OE6
- net N$26: now also R6.!1OE8; no longer U$27.!1OE8
- net N$27: now also R6.!1OE6; no longer U$27.!1OE6
- net N$28: now also R6.!1OE4; no longer U$27.!1OE4
- net N$29: now also R6.!1OE2; no longer U$27.!1OE2
- net N$3: now also R4.!1OE4; no longer U$25.!1OE4
- net N$38: now also R7.!1OE8; no longer U$28.!1OE8
- net N$39: now also R7.!1OE6; no longer U$28.!1OE6
- net N$4: now also R4.!1OE2; no longer U$25.!1OE2
- net N$40: now also R7.!1OE4; no longer U$28.!1OE4
- net N$41: now also R7.!1OE2; no longer U$28.!1OE2
- net OUT1: now also Q24.B-IN, R5.!1OE5, R8.22; no longer U$24.B-IN, U$26.!1OE5, U8.22
- net OUT10: now also R13.!1OE1, R6.!1OE5, R9.44; no longer U$20.!1OE1, U$27.!1OE5, U7.44
- net OUT11: now also R12.!1OE3, R7.!1OE7, R9.88; no longer U$19.!1OE3, U$28.!1OE7, U7.88
- net OUT12: now also R12.!1OE7, R6.!1OE3, R9.77; no longer U$19.!1OE7, U$27.!1OE3, U7.77
- net OUT13: now also R12.!1OE5, R6.!1OE1, R9.33; no longer U$19.!1OE5, U$27.!1OE1, U7.33
- net OUT14: now also R12.!1OE1, R7.!1OE5, R9.22; no longer U$19.!1OE1, U$28.!1OE5, U7.22
- net OUT15: now also R11.!1OE7, R7.!1OE3, R9.99; no longer U$21.!1OE7, U$28.!1OE3, U7.99
- net OUT16: now also R11.!1OE5, R7.!1OE1, R9.11; no longer U$21.!1OE5, U$28.!1OE1, U7.11
- net OUT2: now also Q24.A-IN, R5.!1OE7, R8.88; no longer U$24.A-IN, U$26.!1OE7, U8.88
- net OUT3: now also Q23.B-IN, R4.!1OE5, R8.44; no longer U$23.B-IN, U$25.!1OE5, U8.44
- net OUT4: now also Q23.A-IN, R4.!1OE7, R8.66; no longer U$23.A-IN, U$25.!1OE7, U8.66
- net OUT5: now also Q22.B-IN, R4.!1OE1, R8.33; no longer U$22.B-IN, U$25.!1OE1, U8.33
- net OUT6: now also Q22.A-IN, R4.!1OE3, R8.77; no longer U$22.A-IN, U$25.!1OE3, U8.77
- net OUT7: now also R13.!1OE7, R5.!1OE3, R8.99; no longer U$20.!1OE7, U$26.!1OE3, U8.99
- net OUT8: now also R13.!1OE5, R5.!1OE1, R8.11; no longer U$20.!1OE5, U$26.!1OE1, U8.11
- net OUT9: now also R13.!1OE3, R6.!1OE7, R9.66; no longer U$20.!1OE3, U$27.!1OE7, U7.66
- net PWR_FET_G1: now also Q2.G, Q8.D2, R10.88; no longer U$10.G, U$8.D2, U9.88
- net PWR_FET_G2: now also Q1.G, Q8.D1, R10.22; no longer U$16.G, U$8.D1, U9.22
- net PWR_FET_G3: now also Q4.G, Q9.D2, R10.77; no longer U$12.G, U$9.D2, U9.77
- net PWR_FET_G4: now also Q3.G, Q9.D1, R10.33; no longer U$11.G, U$9.D1, U9.33
- net PWR_FET_G5: now also Q15.D2, Q6.G, R10.66; no longer U$14.G, U$15.D2, U9.66
- net PWR_FET_G6: now also Q15.D1, Q5.G, R10.44; no longer U$13.G, U$15.D1, U9.44
- net PWR_P_FET_1: now also Q6.D; no longer U$14.D
- net PWR_P_FET_2: now also Q5.D; no longer U$13.D
- net PWR_P_FET_3: now also Q4.D; no longer U$12.D
- net PWR_P_FET_4: now also Q3.D; no longer U$11.D
- net PWR_P_FET_5: now also Q2.D; no longer U$10.D
- net PWR_P_FET_6: now also Q1.D; no longer U$16.D
- net RX_UART: now also J4.4
- net TX_UART: now also J4.5
Other:
- note added: "12V INPUT"
- note added: "3.3V REGULATOR"
- note added: "ADDR: 0x18"
- note added: "ADDR: 0x20"
- note added: "ADDR: 0x48"
- note added: "GATE PULLUPS"
- note added: "I2C ADC"
- note added: "I2C GPIO EXPANDER"
- note added: "I2C TEMP SENSOR"
- note added: "MOSFET DRIVERS"
- note added: "N-CHAN MOSFET GATE SERIES RES."
- note added: "N-CHAN MOSFETS"
- note added: "OUTPUT PULL DOWNS"
- note added: "OUTPUT STATE LEDS"
- note added: "POWER MOSFETS"
- note added: "RASPI HEADER"
- note added: "SCREW TERMINALS"
- note added: "SERIAL BUS HEADERS"
- note removed: "SERIAL BUSES"
- moved on the sheet: C1, C10, C2, C3, C4, C5, C6, C7, C8, C9, D1, D10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
