File: eb-ground-station/power-system/ground_station_power_board/UPD-board/power_switching.kicad_sch (KiCad schematic)
At the start: 70 parts, among them Q1 DMN61D8L-LVT, Q10 DMN61D8L-LVT, Q11 SUD50P08-25L-E3, Q12 SUD50P08-25L-E3, Q13 DMN61D8L-LVT, Q14 DMN61D8L-LVT, Q15 DMN61D8L-LVT, Q16 SUD50P08-25L-E3, Q17 SUD50P08-25L-E3, Q18 DMN61D8L-LVT, Q19 SUD50P08-25L-E3, Q2 DMN61D8L-LVT, Q20 SUD50P08-25L-E3, Q3 DMN61D8L-LVT, Q4 SUD50P08-25L-E3, Q5 SUD50P08-25L-E3, Q6 DMN61D8L-LVT, Q7 DMN61D8L-LVT, Q8 DMN61D8L-LVT, Q9 DMN61D8L-LVT, U10 TC4427, U11 TC4427, U12 TC4427, U14 TC4427, U15 TC4427, U16 TC4427, U17 TC4427, U9 TC4427

Commit message: Silkscreen almost done
Parts:
- renumbered C15 to C14, C14 to C15, R9 to R10, R10 to R11, R11 to R12, R12 to R13, R13 to R14, R14 to R15, R15 to R16, R16 to R17, R17 to R18, R18 to R19, R19 to R20, R20 to R21, R21 to R22, R22 to R23, R23 to R26, R8 to R9
Changed lines of the file:
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@@
   (symbol (lib_id "Device:R") (at 90.17 35.56 90) (unit 1)
     (in_bom yes) (on_board yes) (fields_autoplaced)
-    (property "Reference" "R8" (id 0) (at 90.17 30.8442 90))
+    (property "Reference" "R9" (id 0) (at 90.17 30.8442 90))
     (property "Value" "10k" (id 1) (at 90.17 33.3811 90))
     (property "Footprint" "Resistor_SMD:R_0603_1608Metric" (id 2) (at 90.17 37.338 90)
@@
   (symbol (lib_id "Device:R") (at 260.35 43.18 90) (unit 1)
     (in_bom yes) (on_board yes) (fields_autoplaced)
-    (property "Reference" "R17" (id 0) (at 260.35 38.4642 90))
+    (property "Reference" "R18" (id 0) (at 260.35 38.4642 90))
     (property "Value" "gate" (id 1) (at 260.35 41.0011 90))
     (property "Footprint" "Resistor_SMD:R_0603_1608Metric" (id 2) (at 260.35 44.958 90)
@@
   (symbol (lib_id "Device:R") (at 90.17 63.5 90) (unit 1)
     (in_bom yes) (on_board yes) (fields_autoplaced)
-    (property "Reference" "R10" (id 0) (at 90.17 58.7842 90))
+    (property "Reference" "R11" (id 0) (at 90.17 58.7842 90))
     (property "Value" "10k" (id 1) (at 90.17 61.3211 90))
     (property "Footprint" "Resistor_SMD:R_0603_1608Metric" (id 2) (at 90.17 65.278 90)
@@
   (symbol (lib_id "Device:R") (at 345.44 71.12 90) (unit 1)
     (in_bom yes) (on_board yes) (fields_autoplaced)
-    (property "Reference" "R23" (id 0) (at 345.44 66.4042 90))
+    (property "Reference" "R26" (id 0) (at 345.44 66.4042 90))
     (property "Value" "gate" (id 1) (at 345.44 68.9411 90))
     (property "Footprint" "Resistor_SMD:R_0603_1608Metric" (id 2) (at 345.44 72.898 90)
@@
   (symbol (lib_id "Device:C") (at 182.245 39.37 0) (unit 1)
     (in_bom yes) (on_board yes) (fields_autoplaced)
-    (property "Reference" "C15" (id 0) (at 185.166 38.5353 0)
+    (property "Reference" "C14" (id 0) (at 185.166 38.5353 0)
       (effects (font (size 1.27 1.27)) (justify left))
     )
@@
   (symbol (lib_id "Device:R") (at 345.44 63.5 90) (unit 1)
     (in_bom yes) (on_board yes) (fields_autoplaced)
-    (property "Reference" "R22" (id 0) (at 345.44 58.7842 90))
+    (property "Reference" "R23" (id 0) (at 345.44 58.7842 90))
     (property "Value" "10k" (id 1) (at 345.44 61.3211 90))
     (property "Footprint" "Resistor_SMD:R_0603_1608Metric" (id 2) (at 345.44 65.278 90)
@@
   (symbol (lib_id "Device:R") (at 175.26 63.5 90) (unit 1)
     (in_bom yes) (on_board yes) (fields_autoplaced)
-    (property "Reference" "R14" (id 0) (at 175.26 58.7842 90))
+    (property "Reference" "R15" (id 0) (at 175.26 58.7842 90))
     (property "Value" "10k" (id 1) (at 175.26 61.3211 90))
     (property "Footprint" "Resistor_SMD:R_0603_1608Metric" (id 2) (at 175.26 65.278 90)
@@
   (symbol (lib_id "Device:R") (at 345.44 43.18 90) (unit 1)
     (in_bom yes) (on_board yes) (fields_autoplaced)
-    (property "Reference" "R21" (id 0) (at 345.44 38.4642 90))
+    (property "Reference" "R22" (id 0) (at 345.44 38.4642 90))
     (property "Value" "gate" (id 1) (at 345.44 41.0011 90))
     (property "Footprint" "Resistor_SMD:R_0603_1608Metric" (id 2) (at 345.44 44.958 90)
@@
   (symbol (lib_id "Device:R") (at 260.35 35.56 90) (unit 1)
     (in_bom yes) (on_board yes) (fields_autoplaced)
-    (property "Reference" "R16" (id 0) (at 260.35 30.8442 90))
+    (property "Reference" "R17" (id 0) (at 260.35 30.8442 90))
     (property "Value" "10k" (id 1) (at 260.35 33.3811 90))
     (property "Footprint" "Resistor_SMD:R_0603_1608Metric" (id 2) (at 260.35 37.338 90)
@@
   (symbol (lib_id "Device:R") (at 90.17 43.18 90) (unit 1)
     (in_bom yes) (on_board yes) (fields_autoplaced)
-    (property "Reference" "R9" (id 0) (at 90.17 38.4642 90))
+    (property "Reference" "R10" (id 0) (at 90.17 38.4642 90))
     (property "Value" "gate" (id 1) (at 90.17 41.0011 90))
     (property "Footprint" "Resistor_SMD:R_0603_1608Metric" (id 2) (at 90.17 44.958 90)
@@
   (symbol (lib_id "Device:R") (at 260.35 71.12 90) (unit 1)
     (in_bom yes) (on_board yes) (fields_autoplaced)
-    (property "Reference" "R19" (id 0) (at 260.35 66.4042 90))
+    (property "Reference" "R20" (id 0) (at 260.35 66.4042 90))
     (property "Value" "gate" (id 1) (at 260.35 68.9411 90))
     (property "Footprint" "Resistor_SMD:R_0603_1608Metric" (id 2) (at 260.35 72.898 90)
@@
   (symbol (lib_id "Device:R") (at 175.26 43.18 90) (unit 1)
     (in_bom yes) (on_board yes) (fields_autoplaced)
-    (property "Reference" "R13" (id 0) (at 175.26 38.4642 90))
+    (property "Reference" "R14" (id 0) (at 175.26 38.4642 90))
     (property "Value" "gate" (id 1) (at 175.26 41.0011 90))
     (property "Footprint" "Resistor_SMD:R_0603_1608Metric" (id 2) (at 175.26 44.958 90)
@@
   (symbol (lib_id "Device:R") (at 260.35 63.5 90) (unit 1)
     (in_bom yes) (on_board yes) (fields_autoplaced)
-    (property "Reference" "R18" (id 0) (at 260.35 58.7842 90))
+    (property "Reference" "R19" (id 0) (at 260.35 58.7842 90))
     (property "Value" "10k" (id 1) (at 260.35 61.3211 90))
     (property "Footprint" "Resistor_SMD:R_0603_1608Metric" (id 2) (at 260.35 65.278 90)
@@
   (symbol (lib_id "Device:R") (at 345.44 35.56 90) (unit 1)
     (in_bom yes) (on_board yes) (fields_autoplaced)
-    (property "Reference" "R20" (id 0) (at 345.44 30.8442 90))
+    (property "Reference" "R21" (id 0) (at 345.44 30.8442 90))
     (property "Value" "10k" (id 1) (at 345.44 33.3811 90))
     (property "Footprint" "Resistor_SMD:R_0603_1608Metric" (id 2) (at 345.44 37.338 90)
@@
   (symbol (lib_id "Device:R") (at 175.26 35.56 90) (unit 1)
     (in_bom yes) (on_board yes) (fields_autoplaced)
-    (property "Reference" "R12" (id 0) (at 175.26 30.8442 90))
+    (property "Reference" "R13" (id 0) (at 175.26 30.8442 90))
     (property "Value" "10k" (id 1) (at 175.26 33.3811 90))
     (property "Footprint" "Resistor_SMD:R_0603_1608Metric" (id 2) (at 175.26 37.338 90)
@@
   (symbol (lib_id "Device:R") (at 175.26 71.12 90) (unit 1)
     (in_bom yes) (on_board yes) (fields_autoplaced)
-    (property "Reference" "R15" (id 0) (at 175.26 66.4042 90))
+    (property "Reference" "R16" (id 0) (at 175.26 66.4042 90))
     (property "Value" "gate" (id 1) (at 175.26 68.9411 90))
     (property "Footprint" "Resistor_SMD:R_0603_1608Metric" (id 2) (at 175.26 72.898 90)
@@
   (symbol (lib_id "Device:R") (at 90.17 71.12 90) (unit 1)
     (in_bom yes) (on_board yes) (fields_autoplaced)
-    (property "Reference" "R11" (id 0) (at 90.17 66.4042 90))
+    (property "Reference" "R12" (id 0) (at 90.17 66.4042 90))
     (property "Value" "gate" (id 1) (at 90.17 68.9411 90))
     (property "Footprint" "Resistor_SMD:R_0603_1608Metric" (id 2) (at 90.17 72.898 90)
@@
   (symbol (lib_id "Device:C") (at 181.61 67.31 0) (unit 1)
     (in_bom yes) (on_board yes) (fields_autoplaced)
-    (property "Reference" "C14" (id 0) (at 184.531 66.4753 0)
-      (effects (font (size 1.27 1.27)) (justify left))
-    )
+    (property "Reference" "C15" (id 0) (at 184.531 66.4753 0)
+      (effects (font (size 1.27 1.27)) (justify left))
+    )

Commit message: Fixed issues discovered during the design review
Parts:
- removed Q10, Q13, Q2, Q6, Q7, Q9: DMN61D8L-LVT, oresat-footprints:TSOT26-6, symbol OreSat-q-mosfet-DMN61D8L-LVT:DMN61D8L-LVT
- added C21, C22, C23, C24, C25, C26, C27, C28: 0.1uf, Capacitor_SMD:C_0603_1608Metric, symbol Device:C
- added unit 2 of Q1
- added unit 2 of Q10
- added unit 2 of Q13
- added unit 2 of Q14
- added Q15, Q16, Q17, Q18, Q19, Q20: DMN61D8L-LVT, oresat-footprints:TSOT26-6, symbol OreSat-q-mosfet-DMN61D8L-LVT:DMN61D8L-LVT
- added unit 2 of Q4
- added unit 2 of Q7
- added RN1, RN2, RN3, RN4, RN5, RN6: 10k, Resistor_SMD:R_Array_Convex_4x0603, symbol Device:R_Pack04
- R10, R11, R12, R13, R14, R15, R16, R17, R18, R19, R20, R21, R22, R23, R26, R9: symbol Device:R -> Device:R_US
- renumbered Q3 to Q1, Q18 to Q10, Q19 to Q11, Q20 to Q12, Q1 to Q13, Q4 to Q2, Q5 to Q3, Q8 to Q4, Q11 to Q5, Q12 to Q6, Q15 to Q7, Q16 to Q8, Q17 to Q9
Connections:
- net +12V: now also C21.1, C22.1, C23.1, C24.1, C25.1, C26.1, C27.1, C28.1
- net CTL_A0: now also RN1.5 (R4.2)
- net CTL_A1: now also RN1.6 (R3.2)
- net CTL_A2: now also RN1.7 (R2.2)
- net CTL_A3: now also RN1.8 (R1.2)
- net CTL_A4: now also RN2.5 (R4.2)
- net CTL_A5: now also RN2.6 (R3.2)
- net CTL_A6: now also RN2.7 (R2.2)
- net CTL_A7: now also RN2.8 (R1.2)
- net CTL_B0: now also RN3.5 (R4.2)
- net CTL_B1: now also RN3.6 (R3.2)
- net CTL_B2: now also RN3.7 (R2.2)
- net CTL_B3: now also RN3.8 (R1.2)
- net CTL_B4: now also RN4.5 (R4.2)
- net CTL_B5: now also RN4.6 (R3.2)
- net CTL_B6: now also RN4.7 (R2.2)
- net CTL_B7: now also RN4.8 (R1.2)
- net CTL_C0: now also RN5.5 (R4.2)
- net CTL_C1: now also RN5.6 (R3.2)
- net CTL_C2: now also RN5.7 (R2.2)
- net CTL_C3: now also RN5.8 (R1.2)
- net CTL_C4: now also RN6.5 (R4.2)
- net CTL_C5: now also RN6.6 (R3.2)
- net CTL_C6: now also RN6.7 (R2.2)
- net CTL_C7: now also RN6.8 (R1.2)
- net GND: now also C21.2, C22.2, C23.2, C24.2, C25.2, C26.2, C27.2, C28.2, Q1.4 (S), Q10.4 (S), Q13.4 (S), Q14.4 (S), Q15.1 (S), Q15.4 (S), Q16.1 (S), Q16.4 (S), Q17.1 (S), Q17.4 (S), Q18.1 (S), Q18.4 (S), Q19.1 (S), Q19.4 (S), Q20.1 (S), Q20.4 (S), Q4.4 (S), Q7.4 (S), RN1.1 (R1.1), RN1.2 (R2.1), RN1.3 (R3.1), RN1.4 (R4.1), RN2.1 (R1.1), RN2.2 (R2.1), RN2.3 (R3.1), RN2.4 (R4.1), RN3.1 (R1.1), RN3.2 (R2.1), RN3.3 (R3.1), RN3.4 (R4.1), RN4.1 (R1.1), RN4.2 (R2.1), RN4.3 (R3.1), RN4.4 (R4.1), RN5.1 (R1.1), RN5.2 (R2.1), RN5.3 (R3.1), RN5.4 (R4.1), RN6.1 (R1.1), RN6.2 (R2.1), RN6.3 (R3.1), RN6.4 (R4.1); no longer Q1.4 (S), Q10.4 (S), Q13.4 (S), Q14.4 (S), Q4.4 (S), Q7.4 (S)
- net MOS_A1: now also Q1.5 (G); no longer Q1.5 (G)
- net MOS_A3: now also Q4.5 (G); no longer Q4.5 (G)
- net MOS_A5: now also Q7.5 (G); no longer Q7.5 (G)
- net MOS_A7: now also Q10.5 (G); no longer Q10.5 (G)
- net MOS_B1: now also Q13.5 (G); no longer Q13.5 (G)
- net MOS_B2: now also Q14.2 (G)
- net MOS_B3: now also Q14.5 (G)
- net MOS_B4: now also Q15.2 (G)
- net MOS_B5: now also Q15.5 (G)
- net MOS_B6: now also Q16.2 (G)
- net MOS_B7: now also Q16.5 (G)
- net MOS_C0: now also Q17.2 (G)
- net MOS_C1: now also Q17.5 (G)
- net MOS_C2: now also Q18.2 (G)
- net MOS_C3: now also Q18.5 (G)
- net MOS_C4: now also Q19.2 (G)
- net MOS_C5: now also Q19.5 (G)
- net MOS_C6: now also Q20.2 (G); no longer Q14.2 (G)
- net MOS_C7: now also Q20.5 (G); no longer Q14.5 (G)
- net OUT_B1: now also Q13.6 (D); no longer Q13.6 (D)
- net OUT_B2: now also Q14.3 (D)
- net OUT_B3: now also Q14.6 (D)
- net OUT_B4: now also Q15.3 (D)
- net OUT_B5: now also Q15.6 (D)
- net OUT_B6: now also Q16.3 (D)
- net OUT_B7: now also Q16.6 (D)
- net OUT_C0: now also Q17.3 (D)
- net OUT_C1: now also Q17.6 (D)
- net OUT_C2: now also Q18.3 (D)
- net OUT_C3: now also Q18.6 (D)
- net OUT_C4: now also Q19.3 (D)
- net OUT_C5: now also Q19.6 (D)
- net OUT_C6: now also Q20.3 (D); no longer Q14.3 (D)
- net OUT_C7: now also Q20.6 (D); no longer Q14.6 (D)
- net at JP23.1 (A), R19.1, R20.1: now also Q7.6 (D); no longer Q7.6 (D)
- net at JP15.1 (A), R11.1, R12.1: now also Q1.6 (D); no longer Q1.6 (D)
- net at JP27.1 (A), R23.1, R26.1: now also Q10.6 (D); no longer Q10.6 (D)
- net at JP19.1 (A), R15.1, R16.1: now also Q4.6 (D); no longer Q4.6 (D)
Other:
- note added: "+16A"
- note added: "+16A W/ Soft Start"
- note added: "-500mA"
- note added: "12V -500mA or +16A"
- note added: "1k"
- note added: "2pad Jumper"
- note added: "5V -500mA or +16A"
- note added: "5V or 12V -500mA or +16A"
- note added: "680k"
- note added: "Both channels in the pair mmust be configured identically"
- note added: "C"
- note added: "Do not populate any component not specified in the table"
- note added: "Dual Driver"
- note added: "Dual MOSFET"
- note added: "IO Pulldowns"
- note added: "Jump the 3 position jumper to select the voltage (if available)"
- note added: "Jumped"
- note added: "Mode"
- note added: "Open"
- note added: "P MOSFET"
- note added: "Ranges: -500mA +16A"
- note added: "Rgate"
- note added: "Yes"
- note added: "add far too many bypass caps to each of the MOSFET drivers"
- note added: "±1.5A"
- note removed: "Jump the 3 position jumper to select the voltage"
- note removed: "Ranges: -500mA ±1.5A +10A"
- moved on the sheet: C12, C13, C14, C15, C16, C17, C18, C19, JP14, JP15, JP18, JP19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

Commit message: Added UART5 breakout pins
Other:
- company: (none) -> Benjamin Crall
- title: (none) -> Uniclogs Power Distribution Board
Changed lines of the file:
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@@
 (kicad_sch (version 20211123) (generator eeschema)
   (paper "USLedger")
+  (title_block
+    (title "Uniclogs Power Distribution Board")
+    (date "2022-09-06")
+    (rev "2")
+    (company "Benjamin Crall")
+  )
   (junction (at 381 48.26) (diameter 0) (color 0 0 0 0)
   )

Commit message: Preparing to make changes for unavailable parts
Parts:
- C12, C13, C14, C15, C16, C17, C18, C19, C21, C22, C23, C24, C25, C26, C27, C28: Distributor (none) -> DigiKey
- renumbered U14 to U10, U16 to U11, U10 to U12, U12 to U13, U15 to U14, U17 to U15, U9 to U8, U11 to U9
Other:
- title: Uniclogs Power Distribution Board -> UniClOGS Power Distribution Board
Changed lines of the file:
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@@
   (paper "USLedger")
   (title_block
-    (title "Uniclogs Power Distribution Board")
+    (title "UniClOGS Power Distribution Board")
     (date "2022-09-06")
     (rev "2")
@@
       (effects (font (size 1.27 1.27)) hide)
     )
+    (property "Distributor" "DigiKey" (id 7) (at 295.91 44.45 0)
+      (effects (font (size 1.27 1.27)) hide)
+    )
     (pin "1")
     (pin "2")
@@
       (effects (font (size 1.27 1.27)) hide)
     )
+    (property "Distributor" "DigiKey" (id 7) (at 209.55 111.76 0)
+      (effects (font (size 1.27 1.27)) hide)
+    )
     (pin "1")
     (pin "2")
@@
   (symbol (lib_id "OreSat-q-mosfet-driver-TC4427:TC4427") (at 238.76 185.42 0) (unit 1)
     (in_bom yes) (on_board yes) (fields_autoplaced)
-    (property "Reference" "U17" (id 0) (at 240.7794 181.8472 0)
+    (property "Reference" "U15" (id 0) (at 240.7794 181.8472 0)
       (effects (font (size 1.27 1.27)) (justify left))
     )
@@
       (effects (font (size 1.27 1.27)) hide)
     )
+    (property "Distributor" "DigiKey" (id 7) (at 162.56 167.64 0)
+      (effects (font (size 1.27 1.27)) hide)
+    )
     (pin "1")
     (pin "2")
@@
       (effects (font (size 1.27 1.27)) hide)
     )
+    (property "Distributor" "DigiKey" (id 7) (at 125.73 67.31 0)
+      (effects (font (size 1.27 1.27)) hide)
+    )
     (pin "1")
     (pin "2")
@@
   (symbol (lib_id "OreSat-q-mosfet-driver-TC4427:TC4427") (at 97.79 129.54 0) (unit 1)
     (in_bom yes) (on_board yes) (fields_autoplaced)
-    (property "Reference" "U9" (id 0) (at 99.8094 125.9672 0)
+    (property "Reference" "U8" (id 0) (at 99.8094 125.9672 0)
       (effects (font (size 1.27 1.27)) (justify left))
     )
@@
   (symbol (lib_id "OreSat-q-mosfet-driver-TC4427:TC4427") (at 238.76 129.54 0) (unit 1)
     (in_bom yes) (on_board yes) (fields_autoplaced)
-    (property "Reference" "U16" (id 0) (at 240.7794 125.9672 0)
+    (property "Reference" "U11" (id 0) (at 240.7794 125.9672 0)
       (effects (font (size 1.27 1.27)) (justify left))
     )
@@
   (symbol (lib_id "OreSat-q-mosfet-driver-TC4427:TC4427") (at 144.78 129.54 0) (unit 1)
     (in_bom yes) (on_board yes) (fields_autoplaced)
-    (property "Reference" "U11" (id 0) (at 146.7994 125.9672 0)
+    (property "Reference" "U9" (id 0) (at 146.7994 125.9672 0)
       (effects (font (size 1.27 1.27)) (justify left))
     )
@@
   (symbol (lib_id "OreSat-q-mosfet-driver-TC4427:TC4427") (at 191.77 129.54 0) (unit 1)
     (in_bom yes) (on_board yes) (fields_autoplaced)
-    (property "Reference" "U14" (id 0) (at 193.7894 125.9672 0)
+    (property "Reference" "U10" (id 0) (at 193.7894 125.9672 0)
       (effects (font (size 1.27 1.27)) (justify left))
     )
@@
   (symbol (lib_id "OreSat-q-mosfet-driver-TC4427:TC4427") (at 97.79 185.42 0) (unit 1)
     (in_bom yes) (on_board yes) (fields_autoplaced)
-    (property "Reference" "U10" (id 0) (at 99.8094 181.8472 0)
+    (property "Reference" "U12" (id 0) (at 99.8094 181.8472 0)
       (effects (font (size 1.27 1.27)) (justify left))
     )
@@
       (effects (font (size 1.27 1.27)) hide)
     )
+    (property "Distributor" "DigiKey" (id 7) (at 115.57 167.64 0)
+      (effects (font (size 1.27 1.27)) hide)
+    )
     (pin "1")
     (pin "2")
@@
       (effects (font (size 1.27 1.27)) hide)
     )
+    (property "Distributor" "DigiKey" (id 7) (at 162.56 111.76 0)
+      (effects (font (size 1.27 1.27)) hide)
+    )
     (pin "1")
     (pin "2")
@@
       (effects (font (size 1.27 1.27)) hide)
     )
+    (property "Distributor" "DigiKey" (id 7) (at 125.73 44.45 0)
+      (effects (font (size 1.27 1.27)) hide)
+    )
     (pin "1")
     (pin "2")
@@
       (effects (font (size 1.27 1.27)) hide)
     )
+    (property "Distributor" "DigiKey" (id 7) (at 210.82 44.45 0)
+      (effects (font (size 1.27 1.27)) hide)
+    )
     (pin "1")
     (pin "2")
@@
   (symbol (lib_id "OreSat-q-mosfet-driver-TC4427:TC4427") (at 144.78 185.42 0) (unit 1)
     (in_bom yes) (on_board yes) (fields_autoplaced)
-    (property "Reference" "U12" (id 0) (at 146.7994 181.8472 0)
+    (property "Reference" "U13" (id 0) (at 146.7994 181.8472 0)
       (effects (font (size 1.27 1.27)) (justify left))
     )
@@
   (symbol (lib_id "OreSat-q-mosfet-driver-TC4427:TC4427") (at 191.77 185.42 0) (unit 1)
     (in_bom yes) (on_board yes) (fields_autoplaced)
-    (property "Reference" "U15" (id 0) (at 193.7894 181.8472 0)
+    (property "Reference" "U14" (id 0) (at 193.7894 181.8472 0)
       (effects (font (size 1.27 1.27)) (justify left))
     )
@@
       (effects (font (size 1.27 1.27)) hide)
     )
+    (property "Distributor" "DigiKey" (id 7) (at 256.54 111.76 0)
+      (effects (font (size 1.27 1.27)) hide)
+    )
     (pin "1")
     (pin "2")
@@
       (effects (font (size 1.27 1.27)) hide)
     )
+    (property "Distributor" "DigiKey" (id 7) (at 381 72.39 0)
+      (effects (font (size 1.27 1.27)) hide)
+    )
     (pin "1")
     (pin "2")
@@
       (effects (font (size 1.27 1.27)) hide)
     )
+    (property "Distributor" "DigiKey" (id 7) (at 256.54 167.64 0)
+      (effects (font (size 1.27 1.27)) hide)
+    )
     (pin "1")
     (pin "2")
@@
       (effects (font (size 1.27 1.27)) hide)
     )
+    (property "Distributor" "DigiKey" (id 7) (at 381 44.45 0)
+      (effects (font (size 1.27 1.27)) hide)
+    )
     (pin "1")
     (pin "2")
@@
       (effects (font (size 1.27 1.27)) hide)
     )
+    (property "Distributor" "DigiKey" (id 7) (at 209.55 166.37 0)
+      (effects (font (size 1.27 1.27)) hide)
+    )
     (pin "1")
     (pin "2")
@@
       (effects (font (size 1.27 1.27)) hide)
     )
+    (property "Distributor" "DigiKey" (id 7) (at 295.91 72.39 0)
+      (effects (font (size 1.27 1.27)) hide)
+    )
     (pin "1")
     (pin "2")
@@
       (effects (font (size 1.27 1.27)) hide)
     )
+    (property "Distributor" "DigiKey" (id 7) (at 115.57 111.76 0)
+      (effects (font (size 1.27 1.27)) hide)
+    )
     (pin "1")
     (pin "2")
@@
       (effects (font (size 1.27 1.27)) hide)
     )
+    (property "Distributor" "DigiKey" (id 7) (at 210.82 67.31 0)
+      (effects (font (size 1.27 1.27)) hide)
+    )
