File: eb-ground-station/power-system/ground_station_power_board/power_switching.kicad_sch (KiCad schematic)
At the start: 84 parts, among them Q1 DMN61D8L-LVT, Q10 DMN61D8L-LVT, Q11 SUD50P08-25L-E3, Q12 SUD50P08-25L-E3, Q13 DMN61D8L-LVT, Q14 DMN61D8L-LVT, Q15 DMN61D8L-LVT, Q16 DMN61D8L-LVT, Q17 DMN61D8L-LVT, Q18 DMN61D8L-LVT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

Commit message: Fixed UPD board, ready for review and ordering
Parts:
- Q1, Q10, Q13, Q14, Q15, Q16, Q17, Q18, Q19, Q20, Q4, Q7: symbol OreSat-q-mosfet-DMN61D8L-LVT:DMN61D8L-LVT -> oresat-transistors:DMN61D8L-LVT
Connections:
- net GND: now also Q1.1 (S), Q1.4 (S), Q10.1 (S), Q10.4 (S), Q4.1 (S), Q4.4 (S), Q7.1 (S), Q7.4 (S); no longer Q1.1 (S), Q1.4 (S), Q10.1 (S), Q10.4 (S), Q4.1 (S), Q4.4 (S), Q7.1 (S), Q7.4 (S)
- net MOS_A0: now also Q1.5 (G); no longer Q1.2 (G)
- net MOS_A1: now also Q1.2 (G); no longer Q1.5 (G)
- net MOS_A2: now also Q4.5 (G); no longer Q4.2 (G)
- net MOS_A3: now also Q4.2 (G); no longer Q4.5 (G)
- net MOS_A4: now also Q7.5 (G); no longer Q7.2 (G)
- net MOS_A5: now also Q7.2 (G); no longer Q7.5 (G)
- net MOS_A6: now also Q10.5 (G); no longer Q10.2 (G)
- net MOS_A7: now also Q10.2 (G); no longer Q10.5 (G)
- net OUT_B0: now also Q13.6 (D); no longer Q13.3 (D)
- net OUT_B1: now also Q13.3 (D); no longer Q13.6 (D)
- net OUT_B2: now also Q14.6 (D); no longer Q14.3 (D)
- net OUT_B3: now also Q14.3 (D); no longer Q14.6 (D)
- net OUT_B4: now also Q15.6 (D); no longer Q15.3 (D)
- net OUT_B5: now also Q15.3 (D); no longer Q15.6 (D)
- net OUT_B6: now also Q16.6 (D); no longer Q16.3 (D)
- net OUT_B7: now also Q16.3 (D); no longer Q16.6 (D)
- net OUT_C0: now also Q17.6 (D); no longer Q17.3 (D)
- net OUT_C1: now also Q17.3 (D); no longer Q17.6 (D)
- net OUT_C2: now also Q18.6 (D); no longer Q18.3 (D)
- net OUT_C3: now also Q18.3 (D); no longer Q18.6 (D)
- net OUT_C4: now also Q19.6 (D); no longer Q19.3 (D)
- net OUT_C5: now also Q19.3 (D); no longer Q19.6 (D)
- net OUT_C6: now also Q20.6 (D); no longer Q20.3 (D)
- net OUT_C7: now also Q20.3 (D); no longer Q20.6 (D)

Commit message: Fixed pin 1 of expanders being pulldown only
Connections:
- net GND: no longer RN1.4 (R4.1), RN3.4 (R4.1), RN5.4 (R4.1)
- new net +3V3: RN1.4 (R4.1), RN3.4 (R4.1), RN5.4 (R4.1)
Changed lines of the file:
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@@
   (junction (at 158.75 193.04) (diameter 0) (color 0 0 0 0)
   )
+  (junction (at 50.8 167.64) (diameter 0) (color 0 0 0 0)
+  )
   (junction (at 205.74 137.16) (diameter 0) (color 0 0 0 0)
   )
@@
   (junction (at 222.25 55.88) (diameter 0) (color 0 0 0 0)
   )
-  (junction (at 48.26 139.7) (diameter 0) (color 0 0 0 0)
-  )
   (junction (at 284.48 40.64) (diameter 0) (color 0 0 0 0)
   )
@@
   (junction (at 137.16 55.88) (diameter 0) (color 0 0 0 0)
   )
-  (junction (at 48.26 198.12) (diameter 0) (color 0 0 0 0)
-  )
   (junction (at 199.39 48.26) (diameter 0) (color 0 0 0 0)
   )
   (junction (at 110.49 190.5) (diameter 0) (color 0 0 0 0)
   )
-  (junction (at 48.26 167.64) (diameter 0) (color 0 0 0 0)
-  )
   (junction (at 307.34 68.58) (diameter 0) (color 0 0 0 0)
   )
@@
     (stroke (width 0) (type default) (color 0 0 0 0))
   )
-  (wire (pts (xy 48.26 198.12) (xy 48.26 200.66))
-    (stroke (width 0) (type default) (color 0 0 0 0))
-  )
   (wire (pts (xy 27.94 74.93) (xy 30.48 74.93))
     (stroke (width 0) (type default) (color 0 0 0 0))
@@
     (stroke (width 0) (type default) (color 0 0 0 0))
   )
-  (wire (pts (xy 48.26 160.02) (xy 48.26 167.64))
+  (wire (pts (xy 48.26 160.02) (xy 48.26 170.18))
     (stroke (width 0) (type default) (color 0 0 0 0))
   )
@@
     (stroke (width 0) (type default) (color 0 0 0 0))
   )
+  (wire (pts (xy 50.8 198.12) (xy 50.8 167.64))
+    (stroke (width 0) (type default) (color 0 0 0 0))
+  )
   (wire (pts (xy 45.72 185.42) (xy 48.26 185.42))
     (stroke (width 0) (type default) (color 0 0 0 0))
@@
     (stroke (width 0) (type default) (color 0 0 0 0))
   )
-  (wire (pts (xy 45.72 167.64) (xy 48.26 167.64))
-    (stroke (width 0) (type default) (color 0 0 0 0))
-  )
   (wire (pts (xy 125.73 63.5) (xy 137.16 63.5))
     (stroke (width 0) (type default) (color 0 0 0 0))
@@
     (stroke (width 0) (type default) (color 0 0 0 0))
   )
+  (wire (pts (xy 50.8 137.16) (xy 50.8 167.64))
+    (stroke (width 0) (type default) (color 0 0 0 0))
+  )
   (wire (pts (xy 45.72 139.7) (xy 48.26 139.7))
     (stroke (width 0) (type default) (color 0 0 0 0))
@@
     (stroke (width 0) (type default) (color 0 0 0 0))
   )
-  (polyline (pts (xy 50.8 130.81) (xy 50.8 227.33))
+  (polyline (pts (xy 53.34 130.81) (xy 53.34 227.33))
     (stroke (width 0) (type default) (color 0 0 0 0))
   )
@@
     (stroke (width 0) (type default) (color 0 0 0 0))
   )
-  (wire (pts (xy 45.72 198.12) (xy 48.26 198.12))
-    (stroke (width 0) (type default) (color 0 0 0 0))
-  )
   (wire (pts (xy 110.49 190.5) (xy 113.03 190.5))
     (stroke (width 0) (type default) (color 0 0 0 0))
@@
     (stroke (width 0) (type default) (color 0 0 0 0))
   )
-  (polyline (pts (xy 50.8 227.33) (xy 21.59 227.33))
+  (polyline (pts (xy 53.34 227.33) (xy 21.59 227.33))
     (stroke (width 0) (type default) (color 0 0 0 0))
   )
@@
     (stroke (width 0) (type default) (color 0 0 0 0))
   )
-  (wire (pts (xy 48.26 137.16) (xy 48.26 139.7))
-    (stroke (width 0) (type default) (color 0 0 0 0))
-  )
   (wire (pts (xy 40.64 54.61) (xy 43.18 54.61))
     (stroke (width 0) (type default) (color 0 0 0 0))
@@
     (stroke (width 0) (type default) (color 0 0 0 0))
   )
+  (wire (pts (xy 50.8 167.64) (xy 45.72 167.64))
+    (stroke (width 0) (type default) (color 0 0 0 0))
+  )
   (wire (pts (xy 27.94 102.87) (xy 30.48 102.87))
     (stroke (width 0) (type default) (color 0 0 0 0))
@@
     (stroke (width 0) (type default) (color 0 0 0 0))
   )
-  (wire (pts (xy 45.72 137.16) (xy 48.26 137.16))
+  (wire (pts (xy 45.72 137.16) (xy 50.8 137.16))
     (stroke (width 0) (type default) (color 0 0 0 0))
   )
@@
     (stroke (width 0) (type default) (color 0 0 0 0))
   )
-  (polyline (pts (xy 21.59 130.81) (xy 50.8 130.81))
+  (polyline (pts (xy 21.59 130.81) (xy 53.34 130.81))
     (stroke (width 0) (type default) (color 0 0 0 0))
   )
@@
     (stroke (width 0) (type default) (color 0 0 0 0))
   )
-  (wire (pts (xy 48.26 167.64) (xy 48.26 170.18))
-    (stroke (width 0) (type default) (color 0 0 0 0))
-  )
   (wire (pts (xy 45.72 205.74) (xy 48.26 205.74))
     (stroke (width 0) (type default) (color 0 0 0 0))
@@
     (stroke (width 0) (type default) (color 0 0 0 0))
   )
+  (wire (pts (xy 45.72 198.12) (xy 50.8 198.12))
+    (stroke (width 0) (type default) (color 0 0 0 0))
+  )
   (wire (pts (xy 27.94 57.15) (xy 30.48 57.15))
     (stroke (width 0) (type default) (color 0 0 0 0))
@@
     (stroke (width 0) (type default) (color 0 0 0 0))
   )
-  (wire (pts (xy 48.26 190.5) (xy 48.26 198.12))
+  (wire (pts (xy 48.26 190.5) (xy 48.26 200.66))
     (stroke (width 0) (type default) (color 0 0 0 0))
   )
@@
     (pin "2")
   )
+  (symbol (lib_id "power:+3V3") (at 50.8 137.16 0) (unit 1)
+    (in_bom yes) (on_board yes) (fields_autoplaced)
+    (property "Reference" "#PWR0110" (id 0) (at 50.8 140.97 0)
+      (effects (font (size 1.27 1.27)) hide)
+    )
+    (property "Value" "+3V3" (id 1) (at 50.8 132.08 0))
+    (property "Footprint" "" (id 2) (at 50.8 137.16 0)
+      (effects (font (size 1.27 1.27)) hide)
+    )
+    (property "Datasheet" "" (id 3) (at 50.8 137.16 0)
+      (effects (font (size 1.27 1.27)) hide)
+    )
+    (pin "1")
+  )
   (symbol (lib_id "power:GND") (at 365.76 48.26 0) (unit 1)

Commit message: rev2.1 should be done
Other:
- note added: "CHx0 will turn on during boot"
Changed lines of the file:
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@@
+    (effects (font (size 1.27 1.27)) (justify left bottom))
+  )
+  (text "CHx0 will turn on\nduring boot" (at 379.73 121.92 0)
     (effects (font (size 1.27 1.27)) (justify left bottom))
   )

Commit message: updated board changes for bom
Parts:
- C12, C13, C14, C15, C16, C17, C18, C19, Q15, Q16, Q17, Q18, Q19, Q20, U8, U9: now not fitted
- R10, R12, R14, R16, R18, R20, R22, R26: value gate -> 10k
